File: kicad_tht/MCEBlaster.kicad_pcb (KiCad board)
At the start: 2 copper layers, 31.1 x 68.6 mm, 16 parts, among them J1 DB9_Male_MountingHoles, J2 Conn_01x02_Male, J3 DB15_Male_HighDensity_Mountin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, J6 Conn_01x06_Male, SW1 AUTO_ADJUST, SW2 PX_CLK_BTN, U1 74LVC245, U2 RaspberryPi_Pico

Commit message: THT pcb updates
Other:
- net class Default removed
