File: kicad/MCEBlaster.kicad_sch (KiCad schematic)
At the start: 19 parts, among them J1 DB9_Male_MountingHoles, J2 Conn_01x02_Male, J3 DB15_Male_HighDensity_Mountin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, J6 Conn_01x06_Male, U1 74FCT245, U2 RaspberryPi_Pico

Commit message: PCB Rev 0.3
Updates the VGA connector footprint. Should accept both "short" and "long" connectors.
Parts:
- J3: footprint Connector_Dsub:DSUB-15-HD_Female_Horizontal_P2.29x1.98mm_EdgePinOffset3.03mm_Housed_MountingHolesOffset4.94mm -> MCEBlaster:VGA_connector_both_short_and_long
Changed lines of the file:
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@@
   (title_block
     (title "MCEBlaster")
-    (date "2025-06-28")
-    (rev "0.2")
+    (date "2025-08-03")
+    (rev "0.3")
     (company "Scrap Computing")
   )
@@
       (effects (font (size 1.27 1.27)))
     )
-    (property "Footprint" "Connector_Dsub:DSUB-15-HD_Female_Horizontal_P2.29x1.98mm_EdgePinOffset3.03mm_Housed_MountingHolesOffset4.94mm" (at 201.93 72.39 0)
-      (effects (font (size 1.27 1.27)) hide)
-    )
+    (property "Footprint" "MCEBlaster:VGA_connector_both_short_and_long" (at 201.93 72.39 0)
+      (effects (font (size 1.27 1.27)) hide)
+    )
